File: 4ch-driver-v0/4ch-driver-v0.kicad_pcb (KiCad board)
At the start: 2 copper layers, 76.2 x 38.2 mm, 70 parts, among them J1 Barrel_Jack, J2 Screw_Terminal_01x04, J3 Screw_Terminal_01x04, J4 Screw_Terminal_01x02, Q1 2N7002E, Q2 2N7002E, Q3 2N7002E, Q4 2N7002E, U1 DRV104PWP, U2 BD750L2FP3-CE2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

Commit message: fixed screw terminal side
Parts:
- J2: moved to B.Cu
- moved J2 15.2 mm to (172.4, 117.1), turned to 180 degrees
Connections:
- J2 pad 1: /inverted_signal/out4 -> /inverted_signal/out3
- J2 pad 3: /inverted_signal/out3 -> /inverted_signal/out4
Routing:
- net GND: track 135.3 -> 140.8 mm, vias 65 -> 66
- net /inverted_signal/out4: track 18.3 -> 23.3 mm
