File: 4ch-driver-v0/inv_drivers.kicad_sch (KiCad schematic)
At the start: 31 parts, among them J2 Screw_Terminal_01x04

Commit message: fixed screw terminal side
Connections:
- net out3: now also J2.1 (Pin_1); no longer J2.3 (Pin_3)
- net out4: now also J2.3 (Pin_3); no longer J2.1 (Pin_1)
Changed lines of the file:
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@@
     (effects (font (size 1.27 1.27)) (justify left bottom))
   )
-  (label "out3" (at 246.253 76.2 0) (fields_autoplaced)
+  (label "out4" (at 246.253 76.2 0) (fields_autoplaced)
     (effects (font (size 1.27 1.27)) (justify left bottom))
   )
@@
     (effects (font (size 1.27 1.27)) (justify left bottom))
   )
-  (label "out4" (at 246.38 71.12 0) (fields_autoplaced)
+  (label "out3" (at 246.38 71.12 0) (fields_autoplaced)
     (effects (font (size 1.27 1.27)) (justify left bottom))
   )
