File: 8ch-driver-v2/8ch-driver-v2.kicad_pcb (KiCad board)
At the start: 4 copper layers, 76.2 x 75.3 mm, 120 parts, among them J1 Barrel_Jack, J2 Screw_Terminal_01x08, J3 Screw_Terminal_01x08, J4 Screw_Terminal_01x14, Q1 2N7002E, Q2 2N7002E, Q3 2N7002E, Q4 2N7002E, Q5 2N7002E, Q6 2N7002E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

Commit message: progress
Parts:
- removed J2, J3: Screw_Terminal_01x08, TerminalBlock_Phoenix:TerminalBlock_Phoenix_PT-1,5-8-5.0-H_1x08_P5.00mm_Horizontal
- removed J4: Screw_Terminal_01x14, TerminalBlock_Phoenix:TerminalBlock_Phoenix_PT-1,5-14-5.0-H_1x14_P5.00mm_Horizontal
- added U17: FT4232H MINI MODULE, Solenoid_Driver:FT4232H_FTD, F.Cu at (180.7, 76.7)
- added U18: BD33FC0FP, Package_TO_SOT_SMD:TO-252-2, F.Cu at (217.1, 63.7)
- C18, C21: value 0.18uF -> 470pF
- C19, C22: value 470pF -> 10uF; footprint Capacitor_SMD:C_1206_3216Metric -> Capacitor_SMD:C_1210_3225Metric
- C20: value 470pF -> 0.18uF
- C23: value 10uF -> 0.18uF; footprint Capacitor_SMD:C_1210_3225Metric -> Capacitor_SMD:C_1206_3216Metric
- C24: value 10uF -> 470pF; footprint Capacitor_SMD:C_1210_3225Metric -> Capacitor_SMD:C_1206_3216Metric
- D12: value LED -> PMEG10010ELRX; footprint LED_SMD:LED_0805_2012Metric -> Diode_SMD:Nexperia_CFP3_SOD-123W
- D15: value PMEG10010ELRX -> LED; footprint Diode_SMD:Nexperia_CFP3_SOD-123W -> LED_SMD:LED_0805_2012Metric
- R27: value 49R9 -> 4k7
- R29: value 4k7 -> 162k
- R30: value 4k7 -> 191k
- R31: value 4k7 -> 49R9
- R32: value 162k -> 4k7
- R33: value 191k -> 4k7
- renumbered Q5 to Q3, Q3 to Q5
Connections:
- net out1 renamed out01
- net out2 renamed out02
- net out3 renamed out03
- net out4 renamed out04
- net out5 renamed out05
- net out8 renamed out08
- C18 pad 2: /additonal-channels-p2/delay7 -> Net-(U6-BOOT)
- C19 pad 1: GND -> +12V
- C19 pad 2: Net-(U6-BOOT) -> GND
- C20 pad 2: Net-(U7-BOOT) -> /additonal-channels-p2/delay7
- C21 pad 2: /additonal-channels-p2/delay8 -> Net-(U7-BOOT)
- C22 pad 1: GND -> +12V
- C22 pad 2: Net-(U8-BOOT) -> GND
- C23 pad 1: +12V -> GND
- C23 pad 2: GND -> /additonal-channels-p2/delay8
- C24 pad 1: +12V -> GND
- C24 pad 2: GND -> Net-(U8-BOOT)
- D12 pad 1: /additonal-channels-p2/fault7 -> out06
- D12 pad 2: Net-(D12-A) -> GND
- D13 pad 1: /additonal-channels-p2/fault8 -> /additonal-channels-p2/fault7
- D14 pad 1: out6 -> out07
- D15 pad 1: out7 -> /additonal-channels-p2/fault8
- D15 pad 2: GND -> Net-(D15-A)
- Q7 pad 1: /additonal-channels-p2/in_term8 -> /additonal-channels-p2/in_term7
- Q7 pad 3: Net-(D23-K) -> Net-(D24-K)
- Q8 pad 1: /additonal-channels-p2/in_term7 -> /additonal-channels-p2/in_term8
- Q8 pad 3: Net-(D24-K) -> Net-(D23-K)
- R1 pad 1: in1 -> Relay01
- R11 pad 1: in3 -> Relay03
- R16 pad 1: in4 -> Relay04
- R21 pad 1: in5 -> Relay05
- R26 pad 1: in6 -> Relay06
- R26 pad 2: /additonal-channels-p2/in_term6 -> /additonal-channels-p2/in_term5
- R27 pad 1: in7 -> +12V
- R27 pad 2: /additonal-channels-p2/in_term7 -> Net-(D11-A)
- R28 pad 1: +12V -> GND
- R28 pad 2: Net-(D11-A) -> /additonal-channels-p2/in_term5
- R29 pad 2: /additonal-channels-p2/in_term6 -> /additonal-channels-p2/duty6
- R30 pad 1: +12V -> GND
- R30 pad 2: Net-(D12-A) -> /additonal-channels-p2/freq6
- R31 pad 1: GND -> Relay07
- R31 pad 2: /additonal-channels-p2/in_term7 -> /additonal-channels-p2/in_term5
- R32 pad 1: GND -> +12V
- R32 pad 2: /additonal-channels-p2/duty6 -> Net-(D13-A)
- R33 pad 2: /additonal-channels-p2/freq6 -> /additonal-channels-p2/in_term5
- R36 pad 1: in8 -> Relay08
- R36 pad 2: /additonal-channels-p2/in_term8 -> /additonal-channels-p2/in_term5
- R37 pad 2: Net-(D13-A) -> Net-(D15-A)
- R38 pad 2: /additonal-channels-p2/in_term8 -> /additonal-channels-p2/in_term5
- R6 pad 1: in2 -> Relay02
- U1 pad 16: GND -> (no net)
- U1 pad 17: GND -> (no net)
- U1 pad 18: GND -> (no net)
- U1 pad 19: GND -> (no net)
- U1 pad 20: GND -> (no net)
- U1 pad 21: GND -> (no net)
- U2 pad 16: GND -> (no net)
- U2 pad 17: GND -> (no net)
- U2 pad 18: GND -> (no net)
- U2 pad 19: GND -> (no net)
- U2 pad 20: GND -> (no net)
- U2 pad 21: GND -> (no net)
- U3 pad 16: GND -> (no net)
- U3 pad 17: GND -> (no net)
- U3 pad 18: GND -> (no net)
- U3 pad 19: GND -> (no net)
- U3 pad 20: GND -> (no net)
- U3 pad 21: GND -> (no net)
- U4 pad 16: GND -> (no net)
- U4 pad 17: GND -> (no net)
- U4 pad 18: GND -> (no net)
- U4 pad 19: GND -> (no net)
- U4 pad 20: GND -> (no net)
- U4 pad 21: GND -> (no net)
- U5 pad 16: GND -> (no net)
- U5 pad 17: GND -> (no net)
- U5 pad 18: GND -> (no net)
- U5 pad 19: GND -> (no net)
- U5 pad 20: GND -> (no net)
- U5 pad 21: GND -> (no net)
- U6 pad 14: /additonal-channels-p2/in_term6 -> /additonal-channels-p2/in_term5
- U6 pad 16: GND -> (no net)
- U6 pad 17: GND -> (no net)
- U6 pad 18: GND -> (no net)
- U6 pad 19: GND -> (no net)
- U6 pad 20: GND -> (no net)
- U6 pad 21: GND -> (no net)
- U6 pad 6: out6 -> out06
- U6 pad 7: out6 -> out06
- U7 pad 14: /additonal-channels-p2/in_term7 -> /additonal-channels-p2/in_term5
- U7 pad 16: GND -> (no net)
- U7 pad 17: GND -> (no net)
- U7 pad 18: GND -> (no net)
- U7 pad 19: GND -> (no net)
- U7 pad 20: GND -> (no net)
- U7 pad 21: GND -> (no net)
- U7 pad 6: out7 -> out07
- U7 pad 7: out7 -> out07
- U8 pad 14: /additonal-channels-p2/in_term8 -> /additonal-channels-p2/in_term5
- U8 pad 16: GND -> (no net)
- U8 pad 17: GND -> (no net)
- U8 pad 18: GND -> (no net)
- U8 pad 19: GND -> (no net)
- U8 pad 20: GND -> (no net)
- U8 pad 21: GND -> (no net)
Routing:
- net Net-(D12-A): track 58.3 -> 0.00 mm
- net (no net): track 0.00 -> 58.3 mm
- net in8: track 53.2 -> 0.00 mm, vias 3 -> 0
- net Relay08: track 0.00 -> 53.2 mm, vias 0 -> 3
- net in1: track 52.2 -> 0.00 mm
- net Relay01: track 0.00 -> 52.2 mm
- net in4: track 51.9 -> 0.00 mm, vias 3 -> 0
- net Relay04: track 0.00 -> 51.9 mm, vias 0 -> 3
- net in5: track 36.4 -> 0.00 mm, vias 1 -> 0
- net Relay05: track 0.00 -> 36.4 mm, vias 0 -> 1
- net in7: track 23.0 -> 0.00 mm, vias 1 -> 0
- net +12V: track 139.4 -> 162.5 mm, vias 25 -> 26
- net in3: track 23.0 -> 0.00 mm, vias 1 -> 0
- net Relay03: track 0.00 -> 23.0 mm, vias 0 -> 1
- net in2: track 17.4 -> 0.00 mm
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
Commit message: mucho mas progresso
Routing:
- net (no net): track 58.3 -> 179.6 mm
- net out06: track 0.00 -> 59.5 mm
- net /additonal-channels-p2/fault7: track 59.5 -> 0.00 mm, vias 2 -> 4
- net out7: track 49.5 -> 0.00 mm, vias 1 -> 0
- net out07: track 0.00 -> 49.5 mm, vias 0 -> 1
- net out6: track 44.8 -> 0.00 mm
- net Net-(D13-A): track 28.5 -> 0.00 mm
- net /additonal-channels-p2/fault8: track 24.5 -> 0.00 mm, vias 2 -> 0
- net /additonal-channels-p2/in_term7: track 16.1 -> 0.00 mm
- net Net-(D23-K): track 51.5 -> 66.3 mm
- net Net-(D24-K): track 14.8 -> 0.00 mm
- net /additonal-channels-p2/in_term6: track 9.92 -> 0.00 mm
- net Net-(D18-A): track 43.0 -> 51.4 mm
- net Net-(D17-A): track 62.0 -> 69.6 mm
- net /additonal-channels-p2/delay7: track 4.38 -> 0.00 mm
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Other:
- board text added: "16Ch_Driver_v2.0"
- board text removed: "8Ch_Driver_v2.0"
